File: smartac_esp32_controller/board/smartac_esp32_controller.kicad_sch (KiCad schematic)
At the start: 15 parts, among them J1 Conn_01x03_Pin, Q1 2N2222A, U1 ESP32-DevKitC

Commit message: Remaping GPIOs: 16 -> 4, 17 -> 5
Connections:
- net GPIO_4: now reaches U1.26 (ADC2_CH0/GPIO4)
- net GPIO_4: now also C5.2, R1.2, R2.1
- net GPIO_5: now reaches U1.29 (GPIO5)
- net GPIO_5: now also R4.1
- removed net GPIO_16: C5.2, R1.2, R2.1, U1.27 (GPIO16)
- net GPIO_17: no longer names the net of U1.28 (GPIO17)
- net GPIO_17: no longer R4.1
Changed lines of the file:
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@@
 	(wire
 		(pts
-			(xy 130.81 120.65) (xy 113.03 120.65)
+			(xy 120.65 72.39) (xy 113.03 72.39)
 		)
 		(stroke
@@
 	(wire
 		(pts
-			(xy 130.81 118.11) (xy 113.03 118.11)
+			(xy 120.65 74.93) (xy 113.03 74.93)
 		)
 		(stroke
@@
 		)
 	)
-	(label "GPIO_16"
+	(label "GPIO_4"
 		(at 162.56 127 180)
 		(effects
@@
 		)
 	)
-	(label "GPIO_17"
+	(label "GPIO_5"
 		(at 161.29 66.04 180)
 		(effects
@@
 		)
 	)
-	(label "GPIO_16"
-		(at 130.81 118.11 0)
+	(label "GPIO_4"
+		(at 120.65 72.39 0)
 		(effects
 			(font
@@
 		)
 	)
-	(label "GPIO_17"
-		(at 130.81 120.65 0)
-		(effects
-			(font
+	(label "GPIO_5"
+		(at 120.65 74.93 0)
+		(effects
+			(font
